File: BMW_E30_Late_Cluster_Nexus/BMW_E30_Late_Cluster_Nexus.kicad_sch (KiCad schematic)
At the start: 19 parts, among them J1 Blue, J2 White, J3 Yellow

Commit message: Updates to Nexus Schematic
C1 - C4 have all pins named. Break wear circuit completed.
Parts:
- added C1, C2: "4N7", symbol Device:C
- added D7, D8: 1N4004, Diode_THT:D_DO-41_SOD81_P10.16mm_Horizontal, symbol Diode:1N4004
- added J4: Conn_01x05_Pin, symbol Connector:Conn_01x05_Pin
- added Q1: BC327, Package_TO_SOT_THT:TO-92_Inline, symbol Transistor_BJT:BC327
- added R10: 10k, symbol Device:R_Small
- added R11: 4k7, symbol Device:R
- added R12: 390R 0W5, symbol Device:R
- added R2: 150R, symbol Device:R
- added R5: 220R 1W, symbol Device:R
- added R9: 10R, symbol Device:R
Connections:
- net Analog speed is gone; now on net Wheel_spd_output: J3.26 (Pin_26)
- net Battery 2 is gone; now on net Charge_ind-: J1.16 (Pin_16), LA12.1 (-)
- net Fuel gauge is gone; now on net Fuel_level: J2.4 (Pin_4), J3.5 (Pin_5)
- net 12V: no longer J1.1 (Pin_1), J1.2 (Pin_2), J1.23 (Pin_23), J1.7 (Pin_7), J2.23 (Pin_23), J2.6 (Pin_6), J3.10 (Pin_10), J3.11 (Pin_11), J3.14 (Pin_14), J3.15 (Pin_15), J3.2 (Pin_2), J3.20 (Pin_20), J3.22 (Pin_22), J3.23 (Pin_23), J3.24 (Pin_24), J3.7 (Pin_7), J3.9 (Pin_9), LA1.1 (-), LA10.1 (-), LA2.1 (-)
- net Check: now also LA3.1 (-); no longer LA3.2 (+)
- net Fog front: no longer J2.22 (Pin_22)
- net Fog rear: no longer J2.14 (Pin_14)
- net Fuel warn: no longer J2.5 (Pin_5), J3.4 (Pin_4)
- net High beam: no longer J1.12 (Pin_12)
- net Oil pressure: no longer J1.18 (Pin_18)
- net Turn L: no longer J2.7 (Pin_7)
- net Turn R: no longer J1.13 (Pin_13)
- net Wheel_spd_output: now reaches J2.10 (Pin_10)
- net Wheel_spd_output: now also J4.2 (Pin_2)
- net Wheel_spd_input: now reaches J2.12 (Pin_12)
- net Wheel_spd_input: now also J4.3 (Pin_3)
- net DKV-DEFEKT: now reaches J2.15 (Pin_15)
- net KL_31h: now reaches J2.19 (Pin_19)
- net N-DKV: now reaches J2.2 (Pin_2)
- net K-DKV: now reaches J2.9 (Pin_9)
- net Fuel_rate_input: now reaches J3.12 (Pin_12)
- net Fuel_rate_input: now also J1.11 (Pin_11), J3.25 (Pin_25)
- net GNDPWR: now reaches J3.16 (Pin_16)
- net GNDPWR: now also J1.20 (Pin_20), J2.16 (Pin_16), J2.21 (Pin_21), J2.3 (Pin_3), J2.8 (Pin_8), J3.1 (Pin_1), J3.19 (Pin_19), J3.3 (Pin_3), J3.6 (Pin_6), LA10.2 (+), LA4.2 (+), LA5.2 (+), LA6.1 (-), LA7.2 (+), LA8.2 (+), J4.4 (Pin_4), R11.1
- net Low_Fuel_ind-: now reaches J3.17 (Pin_17)
- net Low_Fuel_ind-: now also J2.5 (Pin_5), J3.4 (Pin_4)
- net Fuel_level: now reaches J3.18 (Pin_18)
- net +12_T15: now reaches J1.10 (Pin_10)
- net +12_T15: now also J1.19 (Pin_19), J1.23 (Pin_23), J1.6 (Pin_6), J2.6 (Pin_6), J3.14 (Pin_14), J3.15 (Pin_15), J3.2 (Pin_2), LA3.2 (+), C1.1, C2.1, D7.2 (A), R5.1
- net Charge_ind-: now reaches J1.3 (Pin_3)
- net Charge_ind-: now also J4.5 (Pin_5), R2.2
- net Reverse_gear: now reaches J1.8 (Pin_8)
- net 5th_gear: now reaches J1.9 (Pin_9)
- net 5V renamed S-DKV
- net Battery 1 renamed Charge_ind+
- net Charge_ind+: now also R2.1
- net Brake fluid renamed Brake_fluid_ind-
- removed net Brake lining: J1.21 (Pin_21), J2.26 (Pin_26), LA10.2 (+)
- removed net GND: J1.20 (Pin_20), J2.16 (Pin_16), J2.21 (Pin_21), J2.3 (Pin_3), J2.8 (Pin_8), J3.1 (Pin_1), LA3.1 (-), LA4.2 (+), LA5.2 (+), LA6.1 (-), LA7.2 (+), LA8.2 (+)
- net GND lighting renamed Illum-
- net Park brake renamed Park_brake_ind-
- net Park_brake_ind-: no longer J3.19 (Pin_19), J3.6 (Pin_6)
- net R renamed +12_T15_ACC
- net +12_T15_ACC: now also J4.1 (Pin_1)
- net SI reset renamed SI_RST
- net Temp gauge renamed Eng_temp_sensor
- net Temp warn renamed Overheat_ind-
- new net: D7.1 (K), Q1.3 (E)
- new net: C2.2, D8.1 (K), Q1.1 (C), R9.1
- new net: Q1.2 (B), R12.2
- new net: LA10.1 (-), R9.2
- new net +12_Start_T50: D8.2 (A), J1.1 (Pin_1), J3.22 (Pin_22), J3.9 (Pin_9)
- new net +12_T30: J1.2 (Pin_2), J3.10 (Pin_10), J3.23 (Pin_23)
- new net Brake_wear_sig_1: J1.21 (Pin_21), R5.2
- new net Brake_wear_sig_2: C1.2, J2.26 (Pin_26), R11.2, R12.1
- new net Engine_spd_input: J3.11 (Pin_11), J3.24 (Pin_24), R10.1
- new net Fog_ind+: J2.22 (Pin_22)
- new net High_beam_ind: J1.12 (Pin_12)
- new net Illum+: J2.23 (Pin_23), J3.20 (Pin_20), J3.7 (Pin_7), LA1.1 (-), LA2.1 (-)
- new net LH_ind: J2.7 (Pin_7)
- new net OIl_pressure_ind-: J1.18 (Pin_18)
- new net RH_ind: J1.13 (Pin_13)
- new net Raw_RPM_input: J1.7 (Pin_7), R10.2
- new net Rear_fog_ind+: J2.14 (Pin_14)
- no-connect marks 0 -> 7
Other:
- title: (none) -> BMW E30 Late Model Cluster Nexus
- moved on the sheet: J1, J2, J3, LA1, LA10, LA11, LA12, LA13, LA14, LA15, LA16, LA2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

Commit message: Nexus Schematic Complete Rough
All connectors are pinned and labeled. Should likely do a double check to verify everything is good and then layout can begin.
Parts:
- removed C1, C2: "4N7", symbol Device:C
- removed D7, D8: 1N4004, Diode_THT:D_DO-41_SOD81_P10.16mm_Horizontal, symbol Diode:1N4004
- removed LA10: Brake pad, mount:B8.5d, symbol Device:Lamp
- removed Q1: BC327, Package_TO_SOT_THT:TO-92_Inline, symbol Transistor_BJT:BC327
- removed R11: 4k7, symbol Device:R
- removed R12: 390R 0W5, symbol Device:R
- removed R5: 220R 1W, symbol Device:R
- removed R9: 10R, symbol Device:R
- added D6, D64: 1N4004, Diode_THT:D_DO-41_SOD81_P10.16mm_Horizontal, symbol Diode:1N4004
- added J5: SI Connector, symbol Connector:Conn_01x19_Socket
- added J6: Tachometer, symbol Connector:Conn_01x10_Socket
- added LA17: Fuel Reserve, mount:B8.5d, symbol Device:Lamp
- added R3: 68R 1W, symbol Device:R
- added U1: Coolant Temp, BMW_Cluster_Connectors:Gauge_fuel_temp, symbol BMW_Cluster_Connectors:Gauge_fuel_temp
- added U2: Fuel Gauge, BMW_Cluster_Connectors:Gauge_fuel_temp, symbol BMW_Cluster_Connectors:Gauge_fuel_temp
- J4: value Conn_01x05_Pin -> Speedometer
- LA13: value Oil pressure -> Oil Pressure
Connections:
- net Fog front is gone; now on net Fog_ind+: LA8.1 (-)
- net Fog rear is gone; now on net Rear_fog_ind+: LA7.1 (-)
- net Fuel warn is gone; now on net Low_Fuel_ind-: LA14.2 (+)
- net High beam is gone; now on net High_beam_ind: LA6.2 (+)
- net Oil pressure is gone; now on net +12_T15: LA13.2 (+)
- net Turn L is gone; now on net LH_ind: LA4.1 (-)
- net Turn R is gone; now on net RH_ind: LA5.1 (-)
- net +12_T15: now also LA11.1 (-), LA14.1 (-), LA15.2 (+), LA9.1 (-), J5.5 (Pin_5), LA17.2 (+), R3.1
- net +12_T30: now also J5.8 (Pin_8), J6.10 (Pin_10)
- net Brake_fluid_ind-: now also D6.2 (A)
- net Charge_ind-: now also D6.1 (K), D64.1 (K)
- net Eng_temp_sensor: now also J5.3 (Pin_3), U1.3 (Vout)
- net Engine_spd_input: now also J5.9 (Pin_9)
- net Fuel_level: now also U2.3 (Vout)
- net Fuel_rate_input: now also J5.10 (Pin_10)
- net GNDPWR: now also J5.7 (Pin_7), J6.9 (Pin_9), U2.2 (GND)
- net Low_Fuel_ind-: now also LA17.1 (-)
- net OIl_pressure_ind-: now also LA13.1 (-)
- net Park_brake_ind-: now also D64.2 (A)
- net SI_RST: now also J5.4 (Pin_4)
- net Wheel_spd_output: now also J5.11 (Pin_11)
- removed net 12V: LA11.1 (-), LA13.1 (-), LA14.1 (-), LA15.2 (+), LA9.1 (-)
- new net: R3.2, U2.1 (Vcc)
- new net EG_1+: J5.15 (Pin_15), J6.5 (Pin_5)
- new net EG_1-: J5.14 (Pin_14), J6.6 (Pin_6)
- new net EG_2+: J5.12 (Pin_12), J6.8 (Pin_8)
- new net EG_2-: J5.13 (Pin_13), J6.7 (Pin_7)
- new net Tach_1+: J5.16 (Pin_16), J6.4 (Pin_4)
- new net Tach_1-: J5.17 (Pin_17), J6.3 (Pin_3)
- new net Tach_2+: J5.18 (Pin_18), J6.2 (Pin_2)
- new net Tach_2-: J5.19 (Pin_19), J6.1 (Pin_1)
- new net Temp_+Ub: J5.1 (Pin_1), U1.1 (Vcc)
- new net Temp_GND: J5.2 (Pin_2), U1.2 (GND)
- no-connect marks 7 -> 8
Other:
- added sheet Brake Wear Circuit (Brake_Wear.kicad_sch)
- moved on the sheet: LA3

Commit message: All Footprints Added to Nexus
All footprints have been added to the nexus board project. Next step is to import them to the layout.
Parts:
- removed LA14: Tank warn, mount:B8.5d, symbol Device:Lamp
- D6: footprint Diode_THT:D_DO-41_SOD81_P10.16mm_Horizontal -> Diode_THT:D_DO-41_SOD81_P12.70mm_Horizontal
- J1: footprint TE_AMP:TE_827881-3 -> BMW_Cluster_Connectors:TE_827881-3
- J2: footprint TE_AMP:TE_827881-2 -> BMW_Cluster_Connectors:TE_827881-2
- J3: footprint TE_AMP:TE_827881-1 -> BMW_Cluster_Connectors:TE_827881-1
- J4: footprint (none) -> BMW_Cluster_Connectors:ConnectorIV_Late
- J5: footprint (none) -> BMW_Cluster_Connectors:ConnectorV_Late
- J6: footprint (none) -> BMW_Cluster_Connectors:Tach_EG_Socket_Late
- LA1, LA2: footprint mount:2821MF -> BMW_Cluster_Connectors:2821MF
- LA11, LA12, LA13, LA15, LA16, LA3, LA4, LA5, LA6, LA7, LA8, LA9: footprint mount:B8.5d -> BMW_Cluster_Connectors:2721MF
- LA14: renamed from LA17; footprint mount:B8.5d -> BMW_Cluster_Connectors:2721MF
- R10: footprint (none) -> Resistor_THT:R_Axial_DIN0207_L6.3mm_D2.5mm_P10.16mm_Horizontal
- R2, R3: footprint (none) -> Resistor_THT:R_Axial_DIN0414_L11.9mm_D4.5mm_P20.32mm_Horizontal
Connections:
- no-connect marks 8 -> 10
Other:
- moved on the sheet: LA16
Changed lines of the file:
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@@
 	)
 	(junction
-		(at 290.83 55.88)
-		(diameter 0)
-		(color 0 0 0 0)
-	)
-	(junction
 		(at 344.17 97.79)
 		(diameter 0)
@@
 	)
 	(no_connect
+		(at 381 100.33)
+	)
+	(no_connect
+		(at 381 110.49)
+	)
+	(no_connect
 		(at 62.23 105.41)
 	)
@@
 	(wire
 		(pts
-			(xy 290.83 55.88) (xy 309.88 55.88)
-		)
-		(stroke
-			(width 0)
-			(type default)
-		)
-	)
-	(wire
-		(pts
 			(xy 144.78 212.09) (xy 113.03 212.09)
 		)
@@
 	(wire
 		(pts
-			(xy 290.83 50.8) (xy 290.83 55.88)
-		)
-		(stroke
-			(width 0)
-			(type default)
-		)
-	)
-	(wire
-		(pts
 			(xy 62.23 40.64) (xy 63.5 40.64)
 		)
@@
 	(wire
 		(pts
-			(xy 309.88 55.88) (xy 309.88 58.42)
-		)
-		(stroke
-			(width 0)
-			(type default)
-		)
-	)
-	(wire
-		(pts
 			(xy 344.17 55.88) (xy 339.09 55.88)
 		)
@@
 	(wire
 		(pts
-			(xy 290.83 55.88) (xy 290.83 58.42)
+			(xy 290.83 50.8) (xy 290.83 58.42)
 		)
 		(stroke
@@
 	(wire
 		(pts
-			(xy 283.21 74.93) (xy 309.88 74.93)
-		)
-		(stroke
-			(width 0)
-			(type default)
-		)
-	)
-	(wire
-		(pts
 			(xy 344.17 97.79) (xy 340.36 97.79)
 		)
@@
 	(wire
 		(pts
-			(xy 309.88 74.93) (xy 309.88 68.58)
-		)
-		(stroke
-			(width 0)
-			(type default)
-		)
-	)
-	(wire
-		(pts
 			(xy 133.35 152.4) (xy 137.16 152.4)
 		)
@@
 		)
 	)
-	(global_label "Low_Fuel_ind-"
-		(shape input)
-		(at 283.21 74.93 180)
-		(fields_autoplaced yes)
-		(effects
-			(font
-				(size 1.27 1.27)
-			)
-			(justify right)
-		)
-		(property "Intersheetrefs" "${INTERSHEET_REFS}"
-			(at 266.3154 74.93 0)
-			(effects
-				(font
-					(size 1.27 1.27)
-				)
-				(justify right)
-				(hide yes)
-			)
-		)
-	)
 	(global_label "Fuel_level"
 		(shape output)
@@
 	)
 	(symbol
-		(lib_id "Device:Lamp")
-		(at 309.88 63.5 180)
-		(unit 1)
-		(exclude_from_sim no)
-		(in_bom yes)
-		(on_board yes)
-		(dnp no)
-		(fields_autoplaced yes)
-		(property "Reference" "LA14"
-			(at 313.69 62.2299 0)
-			(effects
-				(font
-					(size 1.27 1.27)
-				)
-				(justify right)
-			)
-		)
-		(property "Value" "Tank warn"
-			(at 313.69 64.7699 0)
-			(effects
-				(font
-					(size 1.27 1.27)
-				)
-				(justify right)
-			)
-		)
-		(property "Footprint" "mount:B8.5d"
-			(at 309.88 66.04 90)
-			(effects
-				(font
-					(size 1.27 1.27)
-				)
-				(hide yes)
-			)
-		)
-		(property "Datasheet" "~"
-			(at 309.88 66.04 90)
-			(effects
-				(font
-					(size 1.27 1.27)
-				)
-				(hide yes)
-			)
-		)
-		(property "Description" ""
-			(at 309.88 63.5 0)
-			(effects
-				(font
-					(size 1.27 1.27)
-				)
-				(hide yes)
-			)
-		)
-		(pin "1"
-		)
-		(pin "2"
-		)
-		(instances
-			(project "e30-cluster"
-				(path "/b71b56f7-638c-4eba-a8eb-f338b4268b5b"
-					(reference "LA14")
-					(unit 1)
-				)
-			)
-		)
-	)
-	(symbol
 		(lib_id "power:+12V")
 		(at 48.26 31.75 0)
@@
 		(on_board yes)
 		(dnp no)
-		(property "Reference" "LA17"
+		(property "Reference" "LA14"
 			(at 347.98 172.7199 0)
 			(effects
@@
 			)
 		)
-		(property "Footprint" "mount:B8.5d"
+		(property "Footprint" "BMW_Cluster_Connectors:2721MF"
 			(at 344.17 171.45 90)
 			(effects
@@
 			(project "BMW_E30_Late_Cluster_Nexus"
 				(path "/b71b56f7-638c-4eba-a8eb-f338b4268b5b"
-					(reference "LA17")
+					(reference "LA14")
 					(unit 1)
 				)
@@
 			)
 		)
-		(property "Footprint" "mount:B8.5d"
+		(property "Footprint" "BMW_Cluster_Connectors:2721MF"
 			(at 208.28 109.22 90)
 			(effects
@@
 			)
 		)
-		(property "Footprint" ""
+		(property "Footprint" "Resistor_THT:R_Axial_DIN0414_L11.9mm_D4.5mm_P20.32mm_Horizontal"
 			(at 377.698 160.02 90)
 			(effects
@@
 			)
 		)
-		(property "Footprint" ""
+		(property "Footprint" "BMW_Cluster_Connectors:ConnectorIV_Late"
 			(at 38.1 215.9 0)
 			(effects
@@
 			)
 		)
-		(property "Footprint" "mount:B8.5d"
+		(property "Footprint" "BMW_Cluster_Connectors:2721MF"
 			(at 227.33 66.04 90)
 			(effects
@@
 			)
 		)
-		(property "Footprint" ""
+		(property "Footprint" "Resistor_THT:R_Axial_DIN0414_L11.9mm_D4.5mm_P20.32mm_Horizontal"
 			(at 357.632 105.41 90)
 			(effects
@@
 			)
 		)
-		(property "Footprint" "mount:B8.5d"
+		(property "Footprint" "BMW_Cluster_Connectors:2721MF"
 			(at 302.26 109.22 90)
 			(effects
@@
 			)
 		)
-		(property "Footprint" "mount:2821MF"
+		(property "Footprint" "BMW_Cluster_Connectors:2821MF"
 			(at 361.95 66.04 90)
 			(effects
@@
 			)
 		)
-		(property "Footprint" ""
+		(property "Footprint" "Resistor_THT:R_Axial_DIN0207_L6.3mm_D2.5mm_P10.16mm_Horizontal"
 			(at 139.7 152.4 0)
 			(effects
@@
 			)
 		)
-		(property "Footprint" "mount:B8.5d"
+		(property "Footprint" "BMW_Cluster_Connectors:2721MF"
 			(at 246.38 104.14 90)
 			(effects
@@
 			)
 		)
-		(property "Footprint" "mount:2821MF"
+		(property "Footprint" "BMW_Cluster_Connectors:2821MF"
 			(at 344.17 66.04 90)
 			(effects
@@
 			)
 		)
-		(property "Footprint" "mount:B8.5d"
+		(property "Footprint" "BMW_Cluster_Connectors:2721MF"
 			(at 284.48 109.22 90)
 			(effects
@@
 			)
 		)
-		(property "Footprint" "Diode_THT:D_DO-41_SOD81_P10.16mm_Horizontal"
+		(property "Footprint" "Diode_THT:D_DO-41_SOD81_P12.70mm_Horizontal"
 			(at 109.855 68.58 0)
 			(effects
@@
 			)
 		)
-		(property "Footprint" "mount:B8.5d"
+		(property "Footprint" "BMW_Cluster_Connectors:2721MF"
 			(at 265.43 171.45 90)
 			(effects
@@
 			)
 		)
-		(property "Footprint" "mount:B8.5d"
+		(property "Footprint" "BMW_Cluster_Connectors:2721MF"
 			(at 290.83 66.04 90)
 			(effects
@@
 			)
 		)
-		(property "Footprint" "mount:B8.5d"
+		(property "Footprint" "BMW_Cluster_Connectors:2721MF"
 			(at 344.17 102.87 90)
 			(effects
@@
 	(symbol
 		(lib_id "Device:Lamp")
-		(at 389.89 100.33 0)
+		(at 381 105.41 0)
 		(unit 1)
 		(exclude_from_sim no)
@@
 		(fields_autoplaced yes)
 		(property "Reference" "LA16"
-			(at 393.7 99.0599 0)
+			(at 384.81 104.1399 0)
 			(effects
 				(font
@@
 		)
 		(property "Value" "Unused"
-			(at 393.7 101.5999 0)
+			(at 384.81 106.6799 0)
 			(effects
 				(font
@@
 			)
 		)
-		(property "Footprint" "mount:B8.5d"
-			(at 389.89 97.79 90)
+		(property "Footprint" "BMW_Cluster_Connectors:2721MF"
+			(at 381 102.87 90)
 			(effects
 				(font
@@
 		)
 		(property "Datasheet" "~"
-			(at 389.89 97.79 90)
+			(at 381 102.87 90)
 			(effects
 				(font
@@
 		)
 		(property "Description" ""
-			(at 389.89 100.33 0)
+			(at 381 105.41 0)
 			(effects
 				(font
@@
 			)
 		)
-		(property "Footprint" ""
+		(property "Footprint" "BMW_Cluster_Connectors:ConnectorV_Late"
 			(at 107.95 224.79 0)
 			(effects
@@
 			)
 		)
-		(property "Footprint" "TE_AMP:TE_827881-2"
+		(property "Footprint" "BMW_Cluster_Connectors:TE_827881-2"
 			(at 54.61 105.41 0)
 			(effects
@@
 			)
 		)
-		(property "Footprint" "mount:B8.5d"
+		(property "Footprint" "BMW_Cluster_Connectors:2721MF"
 			(at 208.28 60.96 90)
 			(effects
@@
 			)
 		)
-		(property "Footprint" "mount:B8.5d"
+		(property "Footprint" "BMW_Cluster_Connectors:2721MF"
 			(at 247.65 171.45 90)
 			(effects
@@
 			)
 		)
-		(property "Footprint" ""
+		(property "Footprint" "BMW_Cluster_Connectors:Tach_EG_Socket_Late"
 			(at 208.28 231.14 0)
 			(effects
@@
 			)
 		)
-		(property "Footprint" "mount:B8.5d"
+		(property "Footprint" "BMW_Cluster_Connectors:2721MF"
 			(at 227.33 109.22 90)
 			(effects
@@
 			)
 		)
-		(property "Footprint" "TE_AMP:TE_827881-1"
+		(property "Footprint" "BMW_Cluster_Connectors:TE_827881-1"
 			(at 54.61 162.56 0)
 			(effects
@@
 			)
 		)
-		(property "Footprint" "TE_AMP:TE_827881-3"
+		(property "Footprint" "BMW_Cluster_Connectors:TE_827881-3"
 			(at 54.61 53.34 0)
 			(effects
