File: BMW_E30_Late_Cluster_Nexus/BMW_E30_Late_Cluster_Nexus.kicad_sch (KiCad schematic)
At the start: 28 parts, among them J1 Blue, J2 White, J3 Yellow, J4 Speedometer, J5 SI Connector, J6 Tachometer, U1 Coolant Temp, U2 Fuel Gauge

Commit message: Update Connector V
Change Connector V to an updated version that is more accurate to the original pins. Note that depending on Early model updates and subsequent board runs, the outline may have to be moved up by 0.2 mm to match it. Also further adjustments of many connectors may need to be updated slightly for fitment purposes
Parts:
- J5: footprint BMW_Cluster_Connectors:ConnectorV_Late -> BMW_Cluster_Connectors:ConnectorV_Late_V2
Changed lines of the file:
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@@
 			)
 		)
-		(property "Footprint" "BMW_Cluster_Connectors:ConnectorV_Late"
+		(property "Footprint" "BMW_Cluster_Connectors:ConnectorV_Late_V2"
 			(at 107.95 224.79 0)
 			(effects

Commit message: Updated R2 Specs
Parts:
- R2: value 150R -> 150R 1W; Digikey Part # (none) -> A131434CT-ND

Commit message: Update Schematic PDFs
Added updates to schematic pdf documents for consistency
Other:
- company: Reagan Ansel -> Reans
Changed lines of the file:
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@@
 		(date "2025-11-10")
 		(rev "0")
-		(company "Reagan Ansel")
+		(company "Reans")
+		(comment 1 "Reagan Ansel")
 	)
 	(junction
@@
 		)
 		(instances
-			(project ""
+			(project "BMW_E30_Late_Cluster_Nexus"
 				(path "/b71b56f7-638c-4eba-a8eb-f338b4268b5b"
 					(reference "D64")
@@
 		)
 		(instances
-			(project "e30-cluster"
+			(project "BMW_E30_Late_Cluster_Nexus"
 				(path "/b71b56f7-638c-4eba-a8eb-f338b4268b5b"
 					(reference "LA4")
@@
 		)
 		(instances
-			(project ""
+			(project "BMW_E30_Late_Cluster_Nexus"
 				(path "/b71b56f7-638c-4eba-a8eb-f338b4268b5b"
 					(reference "U2")
@@
 		)
 		(instances
-			(project ""
+			(project "BMW_E30_Late_Cluster_Nexus"
 				(path "/b71b56f7-638c-4eba-a8eb-f338b4268b5b"
 					(reference "J4")
@@
 		)
 		(instances
-			(project "e30-cluster"
+			(project "BMW_E30_Late_Cluster_Nexus"
 				(path "/b71b56f7-638c-4eba-a8eb-f338b4268b5b"
 					(reference "LA11")
@@
 		)
 		(instances
-			(project ""
+			(project "BMW_E30_Late_Cluster_Nexus"
 				(path "/b71b56f7-638c-4eba-a8eb-f338b4268b5b"
 					(reference "R2")
@@
 		)
 		(instances
-			(project "e30-cluster"
+			(project "BMW_E30_Late_Cluster_Nexus"
 				(path "/b71b56f7-638c-4eba-a8eb-f338b4268b5b"
 					(reference "LA8")
@@
 		)
 		(instances
-			(project ""
+			(project "BMW_E30_Late_Cluster_Nexus"
 				(path "/b71b56f7-638c-4eba-a8eb-f338b4268b5b"
 					(reference "LA1")
@@
 		)
 		(instances
-			(project ""
+			(project "BMW_E30_Late_Cluster_Nexus"
 				(path "/b71b56f7-638c-4eba-a8eb-f338b4268b5b"
 					(reference "R10")
@@
 		)
 		(instances
-			(project "e30-cluster"
+			(project "BMW_E30_Late_Cluster_Nexus"
 				(path "/b71b56f7-638c-4eba-a8eb-f338b4268b5b"
 					(reference "LA6")
@@
 		)
 		(instances
-			(project ""
+			(project "BMW_E30_Late_Cluster_Nexus"
 				(path "/b71b56f7-638c-4eba-a8eb-f338b4268b5b"
 					(reference "#PWR05")
@@
 		)
 		(instances
-			(project "e30-cluster"
+			(project "BMW_E30_Late_Cluster_Nexus"
 				(path "/b71b56f7-638c-4eba-a8eb-f338b4268b5b"
 					(reference "LA2")
@@
 		)
 		(instances
-			(project "e30-cluster"
+			(project "BMW_E30_Late_Cluster_Nexus"
 				(path "/b71b56f7-638c-4eba-a8eb-f338b4268b5b"
 					(reference "LA7")
@@
 		)
 		(instances
-			(project "e30-cluster"
+			(project "BMW_E30_Late_Cluster_Nexus"
 				(path "/b71b56f7-638c-4eba-a8eb-f338b4268b5b"
 					(reference "LA9")
@@
 		)
 		(instances
-			(project "e30-cluster"
+			(project "BMW_E30_Late_Cluster_Nexus"
 				(path "/b71b56f7-638c-4eba-a8eb-f338b4268b5b"
 					(reference "LA12")
@@
 		)
 		(instances
-			(project ""
+			(project "BMW_E30_Late_Cluster_Nexus"
 				(path "/b71b56f7-638c-4eba-a8eb-f338b4268b5b"
 					(reference "#PWR01")
@@
 		)
 		(instances
-			(project "e30-cluster"
+			(project "BMW_E30_Late_Cluster_Nexus"
 				(path "/b71b56f7-638c-4eba-a8eb-f338b4268b5b"
 					(reference "LA16")
@@
 		)
 		(instances
-			(project ""
+			(project "BMW_E30_Late_Cluster_Nexus"
 				(path "/b71b56f7-638c-4eba-a8eb-f338b4268b5b"
 					(reference "J5")
@@
 		)
 		(instances
-			(project ""
+			(project "BMW_E30_Late_Cluster_Nexus"
 				(path "/b71b56f7-638c-4eba-a8eb-f338b4268b5b"
 					(reference "J2")
@@
 		)
 		(instances
-			(project "e30-cluster"
+			(project "BMW_E30_Late_Cluster_Nexus"
 				(path "/b71b56f7-638c-4eba-a8eb-f338b4268b5b"
 					(reference "LA15")
@@
 		)
 		(instances
-			(project "e30-cluster"
+			(project "BMW_E30_Late_Cluster_Nexus"
 				(path "/b71b56f7-638c-4eba-a8eb-f338b4268b5b"
 					(reference "LA3")
@@
 		)
 		(instances
-			(project ""
+			(project "BMW_E30_Late_Cluster_Nexus"
 				(path "/b71b56f7-638c-4eba-a8eb-f338b4268b5b"
 					(reference "J6")
@@
 		)
 		(instances
-			(project "e30-cluster"
+			(project "BMW_E30_Late_Cluster_Nexus"
 				(path "/b71b56f7-638c-4eba-a8eb-f338b4268b5b"
 					(reference "LA5")
@@
 		)
 		(instances
-			(project ""
+			(project "BMW_E30_Late_Cluster_Nexus"
 				(path "/b71b56f7-638c-4eba-a8eb-f338b4268b5b"
 					(reference "U1")
@@
 		)
 		(instances
-			(project ""
+			(project "BMW_E30_Late_Cluster_Nexus"
 				(path "/b71b56f7-638c-4eba-a8eb-f338b4268b5b"
 					(reference "J3")
@@
 		)
 		(instances
-			(project ""
+			(project "BMW_E30_Late_Cluster_Nexus"
 				(path "/b71b56f7-638c-4eba-a8eb-f338b4268b5b"
 					(reference "J1")
@@
 	)
 	(embedded_fonts no)
+	(embedded_files
+		(file
+			(name "reans_sheet_template.kicad_wks")
+			(type worksheet)
+			(data |KLUv/WD/Cu0XAPbhaSEA1TZqxSYVNDoEMnCBWkUAFLHYT8LfLc64wmSW/n9CwQRfAFoAZABfTlM7
+				Cd4PPZP4H186+DUZmyftazMZJC2P8bFwUWq25kUL8mvHwkXR9pEtP+RPAAACHc97OanDZJkyfiu6
+				ZexMnfGD2a9nCIBAQaOUVnXWvtiW2T8EQKDkgCwiGFoOIdn/etgijP3Ss7lq001Ur56Xy2XSChD4
+				izG0r9ol7kx06g/5X/6a1VV7XqJQDq990Dues9+Mwx979pw4IR4v7ePbb9d8i9eDM9hT/3WSxGHt
+				2uJ1q+pJaX8GA4vQjuDbzqhJOcfXfePbr1LR9rtrPIGhJBC7qR8kM8Z09g4omXCSTTKynjjiS1u1
+				q3CTj080beoGpaw+TAqJdN6Eq1gUW6JrkAYXdfWk9EBhnWkl7tsUFo7ieR1p0Ah/UJFzFgWBwsys
+				itUDRWfNENlvxpauoBUjcUhlrs3u12aulxf0XKs+aBalZRWr16FaFa1zTkqrrWV11qovCsPoB+Ee
+				j0iCNBBdsEPihDapC6udeZCNyxjfJvk4juFpWkVZjw3CObqFDYCaoBFNhdgMSQqSFDLMAYBEhObI
+				NmZkXfEEgg31YlRO4GceOtZZSD4tPZJ8rJ74G8PkjH1JKkKawsKGheoJuP2+IlY18ntrNC2s74Pr
+				DVe+cSgd0L7HteZMeDaXmooSSh/c+bVoVTYLk6RKN7Cv2UoaCAZv6YCSS6nbIQTWD7UwQeis5W/V
+				g0dYgB5CyE6HNFbmmlkm5KySJ6yIRrRM5Uc4pc8u9BJFUDGI5kCOG6xadygVBOu2LFloyz3FUwK0
+				K2QvICvncQgSH7pSFluywCLJ0Rwlm2f0GkYN7sFxT4mPYCI2kaL4bSAlPOhlas5v4CmJJDLxSXKn
+				Odp9OHfwRZI7o8xhC2+Z4AAEWT5Rojog0dbMToQXcXHPsDoOuhAAXPmNnp2jRa7V/EUBa9S+lvzC
+				Ux9y2yG0bmId6AOKOjzjaHSplt4lCml0x3i3uxaxGR+0Cg==|
+			)
+			(checksum "582015C87F5C50DCCFBFE692861C814F")
+		)
+	)
 )
