File: BMW_E30_Late_Cluster_SI/BMW_E30_Late_Cluster_SI.kicad_pcb (KiCad board)
At the start: 2 copper layers, 300 x 53 mm, 103 parts, among them J1 SI LED Board, J2 Coding Plug, J5 Nexus Connector, Q11 BC327-16, Q12 BC337-25, Q13 BC337-16, Q14 BC547B, Q15 BC557B, Q17 BC337-25, Q19 BC337-25, Q21 BC337-25, Q22 BC337-25, Q23 BC337-25, U1 ITT SAF1190-196 MCU, U2 ITT V3003-393, U3 ITT V3004-520, U4 ITT SAF1194-280 MCU, U5 LP2950-5.0_TO92, Y1 Crystal, Y2 Crystal

Commit message: SI Board Layout Complete
Parts:
- added JP1: Jumper, SI_THT:Jumper_THT_P9.7mm, F.Cu at (109.9, 160.3)
- added JP10: Jumper, SI_THT:Jumper_THT_P9.7mm, F.Cu at (170.9, 157.9)
- added JP11: Jumper, SI_THT:Jumper_THT_P9.7mm, F.Cu at (188.7, 148.2)
- added JP12: Jumper, SI_THT:Jumper_THT_P9.7mm, F.Cu at (178.6, 179.1)
- added JP2: Jumper, SI_THT:Jumper_THT_P9.7mm, F.Cu at (145.5, 148.6)
- added JP3: Jumper, SI_THT:Jumper_THT_P9.7mm, F.Cu at (148.0, 148.6)
- added JP4: Jumper, SI_THT:Jumper_THT_P9.7mm, F.Cu at (154.2, 164.9)
- added JP5: Jumper, SI_THT:Jumper_THT_P9.7mm, F.Cu at (154.2, 152.6)
- added JP6: Jumper, SI_THT:Jumper_THT_P9.7mm, F.Cu at (156.2, 155.2)
- added JP7: Jumper, SI_THT:Jumper_THT_P9.7mm, F.Cu at (156.2, 152.6)
- added JP8: Jumper, SI_THT:Jumper_THT_P9.7mm, F.Cu at (158.7, 155.2)
- added JP9: Jumper, SI_THT:Jumper_THT_P9.7mm, F.Cu at (158.7, 142.9)
- C11: footprint Capacitor_THT:CP_Radial_Tantal_D9.0mm_P2.50mm -> Capacitor_THT:CP_Radial_Tantal_D8.0mm_P2.50mm
- moved U4 1.69 mm to (99.7, 172.8)
- moved C21 1.68 mm to (85.8, 155.0)
- moved D26 1.68 mm to (91.4, 155.1)
- moved R46 1.68 mm to (92.8, 151.5)
- moved Y2 1.10 mm to (115.0, 177.6)
- moved C13 1.10 mm to (89.0, 175.8)
- moved C11 0.85 mm to (99.8, 177.3)
- moved Q14 0.80 mm to (107.0, 177.5)
- moved C14 0.51 mm to (127.8, 180.4)
- renumbered JP1 to JP20
Connections:
- C10 pad 1: IC3_P7 -> IC2_P1
- C14 pad 1: Net-(C14-Pad1) -> Net-(JP1-B)
- JP20 pad 1: +5V -> Net-(JP12-B)
- R29 pad 2: Net-(C14-Pad1) -> Net-(JP1-B)
- R45 pad 1: IC2_P12 -> Net-(JP8-B)
- R45 pad 2: IC2_P11 -> Net-(JP6-B)
- U1 pad 21: GNDPWR -> Net-(JP3-B)
- U1 pad 22: IC1_P22 -> Net-(JP2-B)
- U1 pad 35: IC1_P35 -> Net-(JP11-B)
- U2 pad 1: IC3_P7 -> IC2_P1
- U3 pad 22: unconnected-(U3-Pad22) -> GNDPWR
- U4 pad 36: Net-(C14-Pad1) -> Net-(JP1-A)
- Y1 pad 1: IC2_P12 -> Net-(JP8-B)
- Y1 pad 2: IC2_P11 -> Net-(JP6-B)
Routing:
- net GNDPWR: track 262.3 -> 766.5 mm, vias 2 -> 24
- net -BATT: track 0.00 -> 312.4 mm, vias 0 -> 1
- net Net-(C14-Pad1): track 305.3 -> 0.00 mm, vias 3 -> 0
- net Net-(JP1-B): track 0.00 -> 288.7 mm, vias 0 -> 1
- net IC1_P22: track 9.85 -> 262.2 mm, vias 0 -> 2
- net +5V: track 204.1 -> 414.5 mm, vias 2 -> 5
- net IC1_P3: track 140.3 -> 320.4 mm, vias 0 -> 1
- net Net-(D1-K): track 130.9 -> 308.1 mm
- net Net-(Q17-C): track 127.4 -> 303.7 mm, vias 1 -> 2
- net IC1_P4: track 144.1 -> 318.7 mm, vias 0 -> 1
- net IC1_P2: track 124.5 -> 295.8 mm, vias 0 -> 1
- net IC4_P40: track 65.2 -> 227.8 mm, vias 1 -> 3
- net Fuel_rate_input: track 0.00 -> 142.3 mm, vias 0 -> 1
- net IC3_P7: track 0.00 -> 138.7 mm, vias 0 -> 2
- net Wheel_spd_output: track 0.00 -> 135.3 mm, vias 0 -> 1
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Other:
- board text added: "Bestü.-Seite"
- board text added: "Lötseite"
- board text added: "ON"
