File: BMW_E30_Late_Cluster_SI/Indicator_Lights.kicad_sch (KiCad schematic)
At the start: 22 parts, among them J1 SI LED Board, Q19 BC337-25, Q21 BC337-25, Q22 BC337-25, Q23 BC337-25, U4 ITT SAF1194-280 MCU, Y2 Crystal

Commit message: Update Schematic PDFs
Added updates to schematic pdf documents for consistency
Other:
- company: Reagan Ansel -> Reans
Changed lines of the file:
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@@
 	(title_block
 		(title "Indicator Lights")
-		(rev "0")
-		(company "Reagan Ansel")
+		(rev "2")
+		(company "Reans")
+		(comment 1 "Reagan Ansel")
+		(comment 2 "Reagan Ansel")
 	)
 	(text "Oil Service Lamp"

Commit message: Update schematic
Change "battery charging" to "Memory Battery Backup" to reflect how the circuit works
Other:
- title: Indicator Lights -> BMW E30 Late Model SI Board
Changed lines of the file:
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@@
 	(paper "A4")
 	(title_block
-		(title "Indicator Lights")
+		(title "BMW E30 Late Model SI Board")
+		(date "2026-06-03")
 		(rev "2")
 		(company "Reans")
 		(comment 1 "Reagan Ansel")
-		(comment 2 "Reagan Ansel")
 	)
 	(text "Oil Service Lamp"
