File: BMW_E30_Late_Cluster_SI/Temperature_Sensor.kicad_sch (KiCad schematic)
At the start: 30 parts, among them Q11 BC327-16, Q12 BC337-25, Q13 BC337-16, Q14 BC547B, Q15 BC557B, Q17 BC337-25

Commit message: Add SMD Provisions
Added SMD mount options for C12, C4, and C2 so that axial lead electrolytics are not necessary to purchase from the BOM.
Parts:
- added C12.1: 100u, Capacitor_SMD:CP_Elec_6.3x5.8, symbol Device:C_Polarized
- C12: now not fitted
Connections:
- net GNDPWR: now also C12.1.2
- net at C12.1, Q17.1 (C), R27.2: now also C12.1.1
Changed lines of the file:
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@@
 		)
 	)
+	(text_box "C12.1 is an SMD provision"
+		(exclude_from_sim no)
+		(at 260.35 57.15 0)
+		(size 17.78 5.08)
+		(margins 0.9525 0.9525 0.9525 0.9525)
+		(stroke
+			(width 0)
+			(type solid)
+		)
+		(fill
+			(type none)
+		)
+		(effects
+			(font
+				(size 1.27 1.27)
+			)
+			(justify left top)
+		)
+	)
 	(junction
 		(at 95.25 43.18)
@@
 	)
 	(junction
+		(at 261.62 80.01)
+		(diameter 0)
+		(color 0 0 0 0)
+	)
+	(junction
 		(at 81.28 43.18)
 		(diameter 0)
@@
 	)
 	(junction
+		(at 261.62 66.04)
+		(diameter 0)
+		(color 0 0 0 0)
+	)
+	(junction
 		(at 77.47 106.68)
 		(diameter 0)
@@
 	(wire
 		(pts
+			(xy 261.62 80.01) (xy 261.62 82.55)
+		)
+		(stroke
+			(width 0)
+			(type default)
+		)
+	)
+	(wire
+		(pts
 			(xy 243.84 118.11) (xy 243.84 123.19)
 		)
@@
 	(wire
 		(pts
+			(xy 274.32 71.12) (xy 274.32 66.04)
+		)
+		(stroke
+			(width 0)
+			(type default)
+		)
+	)
+	(wire
+		(pts
 			(xy 162.56 55.88) (xy 162.56 62.23)
 		)
@@
 	(wire
 		(pts
-			(xy 266.7 78.74) (xy 266.7 82.55)
+			(xy 261.62 78.74) (xy 261.62 80.01)
 		)
 		(stroke
@@
 	(wire
 		(pts
-			(xy 266.7 66.04) (xy 266.7 71.12)
+			(xy 261.62 66.04) (xy 261.62 71.12)
 		)
 		(stroke
@@
 	(wire
 		(pts
-			(xy 243.84 66.04) (xy 266.7 66.04)
+			(xy 243.84 66.04) (xy 261.62 66.04)
 		)
 		(stroke
@@
 	(wire
 		(pts
+			(xy 274.32 78.74) (xy 274.32 80.01)
+		)
+		(stroke
+			(width 0)
+			(type default)
+		)
+	)
+	(wire
+		(pts
 			(xy 77.47 124.46) (xy 109.22 124.46)
 		)
@@
 	(wire
 		(pts
+			(xy 274.32 80.01) (xy 261.62 80.01)
+		)
+		(stroke
+			(width 0)
+			(type default)
+		)
+	)
+	(wire
+		(pts
 			(xy 93.98 168.91) (xy 48.26 168.91)
 		)
@@
 	(wire
 		(pts
+			(xy 274.32 66.04) (xy 261.62 66.04)
+		)
+		(stroke
+			(width 0)
+			(type default)
+		)
+	)
+	(wire
+		(pts
 			(xy 116.84 173.99) (xy 116.84 177.8)
 		)
@@
 	)
 	(symbol
+		(lib_id "Device:C_Polarized")
+		(at 274.32 74.93 0)
+		(unit 1)
+		(exclude_from_sim no)
+		(in_bom yes)
+		(on_board yes)
+		(dnp no)
+		(fields_autoplaced yes)
+		(property "Reference" "C12.1"
+			(at 278.13 72.7709 0)
+			(effects
+				(font
+					(size 1.27 1.27)
+				)
+				(justify left)
+			)
+		)
+		(property "Value" "100u"
+			(at 278.13 75.3109 0)
+			(effects
+				(font
+					(size 1.27 1.27)
+				)
+				(justify left)
+			)
+		)
+		(property "Footprint" "Capacitor_SMD:CP_Elec_6.3x5.8"
+			(at 275.2852 78.74 0)
+			(effects
+				(font
+					(size 1.27 1.27)
+				)
+				(hide yes)
+			)
+		)
+		(property "Datasheet" "https://www.nichicon.co.jp/english/series_items/catalog_pdf/e-ucd.pdf"
+			(at 274.32 74.93 0)
+			(effects
+				(font
+					(size 1.27 1.27)
+				)
+				(hide yes)
+			)
+		)
+		(property "Description" "16v"
+			(at 274.32 74.93 0)
+			(effects
+				(font
+					(size 1.27 1.27)
+				)
+				(hide yes)
+			)
+		)
+		(property "Vendor Link" "https://www.digikey.com/en/products/detail/nichicon/UCD1C101MCL1GS/2549642"
+			(at 274.32 74.93 0)
+			(effects
+				(font
+					(size 1.27 1.27)
+				)
+				(hide yes)
+			)
+		)
+		(pin "2"
+		)
+		(pin "1"
+		)
+		(instances
+			(project "BMW_E30_Late_Cluster_SI"
+				(path "/00d578f4-1582-4e4e-9a07-e5462d38fb61/84ca9cc6-3e51-42c7-8f6d-11ef7495b962"
+					(reference "C12.1")
+					(unit 1)
+				)
+			)
+		)
+	)
+	(symbol
 		(lib_id "power:GNDPWR")
 		(at 95.25 63.5 0)
@@
 	(symbol
 		(lib_id "power:GNDPWR")
-		(at 266.7 82.55 0)
+		(at 261.62 82.55 0)
 		(unit 1)
 		(exclude_from_sim no)
@@
 		(fields_autoplaced yes)
 		(property "Reference" "#PWR043"
-			(at 266.7 87.63 0)
+			(at 261.62 87.63 0)
 			(effects
 				(font
@@
 		)
 		(property "Value" "GNDPWR"
-			(at 266.573 86.36 0)
+			(at 261.493 86.36 0)
 			(effects
 				(font
@@
 		)
 		(property "Footprint" ""
-			(at 266.7 83.82 0)
+			(at 261.62 83.82 0)
 			(effects
 				(font
@@
 		)
 		(property "Datasheet" ""
-			(at 266.7 83.82 0)
+			(at 261.62 83.82 0)
 			(effects
 				(font
@@
 		)
 		(property "Description" "Power symbol creates a global label with name \"GNDPWR\" , global ground"
-			(at 266.7 82.55 0)
+			(at 261.62 82.55 0)
 			(effects
 				(font
@@
 	(symbol
 		(lib_id "Device:C_Polarized")
-		(at 266.7 74.93 0)
+		(at 261.62 74.93 0)
 		(unit 1)
 		(exclude_from_sim no)
 		(in_bom yes)
 		(on_board yes)
-		(dnp no)
+		(dnp yes)
 		(fields_autoplaced yes)
 		(property "Reference" "C12"
-			(at 270.51 72.7709 0)
+			(at 265.43 72.7709 0)
 			(effects
 				(font
@@
 		)
 		(property "Value" "100u"
-			(at 270.51 75.3109 0)
+			(at 265.43 75.3109 0)
 			(effects
 				(font
@@
 		)
 		(property "Footprint" "Capacitor_THT:CP_Axial_L18.0mm_D6.5mm_P25.00mm_Horizontal"
-			(at 267.6652 78.74 0)
+			(at 262.5852 78.74 0)
 			(effects
 				(font
@@
 		)
 		(property "Datasheet" "~"
-			(at 266.7 74.93 0)
+			(at 261.62 74.93 0)
 			(effects
 				(font
@@
 		)
 		(property "Description" "16v"
-			(at 266.7 74.93 0)
+			(at 261.62 74.93 0)
 			(effects
 				(font
@@
 		)
 		(property "Vendor Link" ""
-			(at 266.7 74.93 0)
+			(at 261.62 74.93 0)
 			(effects
 				(font

Commit message: Update Schematic PDFs
Added updates to schematic pdf documents for consistency
Other:
- company: Reagan Ansel -> Reans
Changed lines of the file:
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@@
 	(title_block
 		(title "Temperature Sensor")
-		(rev "0")
-		(company "Reagan Ansel")
+		(rev "2")
+		(company "Reans")
+		(comment 1 "Reagan Ansel")
+		(comment 2 "Reagan Ansel")
 	)
 	(text_box "Temp_+Ub and Temp_GND provide power to the temperature sensor gauge"

Commit message: Update schematic
Change "battery charging" to "Memory Battery Backup" to reflect how the circuit works
Other:
- title: Temperature Sensor -> BMW E30 Late Model SI Board
Changed lines of the file:
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@@
 	(paper "A4")
 	(title_block
-		(title "Temperature Sensor")
+		(title "BMW E30 Late Model SI Board")
+		(date "2026-06-03")
 		(rev "2")
 		(company "Reans")
 		(comment 1 "Reagan Ansel")
-		(comment 2 "Reagan Ansel")
 	)
 	(text_box "Temp_+Ub and Temp_GND provide power to the temperature sensor gauge"
